Commit message: URDFファイル内のメッシュパスを修正し、環境設定ファイルとトレーニング設定ファイルを追加。報酬関数の設定を修正し、物理パラメータの設定を更新。

File: assets/bittle-urdf/bittle.urdf (robot description, URDF)
Before this commit: robot bittle, 13 links, 12 joints
Links:
- link base-frame-link: geometry collision mesh filename=obj/base_frame.001.obj scale=1.0 1.0 1.0; visual mesh filename=obj/base_frame.obj scale=1.0 1.0 1.0
- link battery-link: geometry collision mesh filename=obj/battery.001.obj scale=1.0 1.0 1.0; visual mesh filename=obj/battery.obj scale=1.0 1.0 1.0
- link cover-link: geometry collision mesh filename=obj/cover.001.obj scale=1.0 1.0 1.0; visual mesh filename=obj/cover.obj scale=1.0 1.0 1.0
- link imu_link: geometry visual mesh filename=obj/Cube.011.obj scale=1.0 1.0 1.0
- link left-back-knee-link: geometry collision mesh filename=obj/left_knee.002.obj scale=1.0 1.0 1.0; visual mesh filename=obj/left_knee.001.obj scale=1.0 1.0 1.0
- link left-back-shoulder-link: geometry collision mesh filename=obj/shoulder.004.obj scale=1.0 1.0 1.0; visual mesh filename=obj/shoulder.001.obj scale=1.0 1.0 1.0
- link left-front-knee-link: geometry collision mesh filename=obj/left_knee.003.obj scale=1.0 1.0 1.0; visual mesh filename=obj/left_knee.obj scale=1.0 1.0 1.0
- link left-front-shoulder-link: geometry collision mesh filename=obj/shoulder.007.obj scale=1.0 1.0 1.0; visual mesh filename=obj/shoulder.obj scale=1.0 1.0 1.0
- link mainboard_link: geometry visual mesh filename=obj/Plane.obj scale=1.0 1.0 1.0
- link right-back-knee-link: geometry collision mesh filename=obj/right_knee.002.obj scale=1.0 1.0 1.0; visual mesh filename=obj/right_knee.001.obj scale=1.0 1.0 1.0
- link right-back-shoulder-link: geometry collision mesh filename=obj/shoulder.005.obj scale=1.0 1.0 1.0; visual mesh filename=obj/shoulder.002.obj scale=1.0 1.0 1.0
- link right-front-knee-link: geometry collision mesh filename=obj/right_knee.003.obj scale=1.0 1.0 1.0; visual mesh filename=obj/right_knee.obj scale=1.0 1.0 1.0
- link right-front-shoulder-link: geometry collision mesh filename=obj/shoulder.006.obj scale=1.0 1.0 1.0; visual mesh filename=obj/shoulder.003.obj scale=1.0 1.0 1.0

Commit message: URDFファイル内のメッシュスケールを0.1に変更し、環境設定ファイルに初期姿勢の多様性設定を追加。報酬関数の改善と学習段階の管理機能を実装。新しい環境設定ファイルとトレーニング設定ファイルを追加し、並列トレーニング用の設定も整備。

File: assets/bittle-urdf/bittle.urdf (robot description, URDF)
Before this commit: robot bittle, 13 links, 12 joints
Links:
- link base-frame-link: geometry collision mesh filename=obj/base_frame.001.obj scale=0.1 0.1 0.1; visual mesh filename=obj/base_frame.obj scale=0.1 0.1 0.1
- link battery-link: geometry collision mesh filename=obj/battery.001.obj scale=0.1 0.1 0.1; visual mesh filename=obj/battery.obj scale=0.1 0.1 0.1
- link cover-link: geometry collision mesh filename=obj/cover.001.obj scale=0.1 0.1 0.1; visual mesh filename=obj/cover.obj scale=0.1 0.1 0.1
- link imu_link: geometry visual mesh filename=obj/Cube.011.obj scale=0.1 0.1 0.1
- link left-back-knee-link: geometry collision mesh filename=obj/left_knee.002.obj scale=0.1 0.1 0.1; visual mesh filename=obj/left_knee.001.obj scale=0.1 0.1 0.1
- link left-back-shoulder-link: geometry collision mesh filename=obj/shoulder.004.obj scale=0.1 0.1 0.1; visual mesh filename=obj/shoulder.001.obj scale=0.1 0.1 0.1
- link left-front-knee-link: geometry collision mesh filename=obj/left_knee.003.obj scale=0.1 0.1 0.1; visual mesh filename=obj/left_knee.obj scale=0.1 0.1 0.1
- link left-front-shoulder-link: geometry collision mesh filename=obj/shoulder.007.obj scale=0.1 0.1 0.1; visual mesh filename=obj/shoulder.obj scale=0.1 0.1 0.1
- link mainboard_link: geometry visual mesh filename=obj/Plane.obj scale=0.1 0.1 0.1
- link right-back-knee-link: geometry collision mesh filename=obj/right_knee.002.obj scale=0.1 0.1 0.1; visual mesh filename=obj/right_knee.001.obj scale=0.1 0.1 0.1
- link right-back-shoulder-link: geometry collision mesh filename=obj/shoulder.005.obj scale=0.1 0.1 0.1; visual mesh filename=obj/shoulder.002.obj scale=0.1 0.1 0.1
- link right-front-knee-link: geometry collision mesh filename=obj/right_knee.003.obj scale=0.1 0.1 0.1; visual mesh filename=obj/right_knee.obj scale=0.1 0.1 0.1
- link right-front-shoulder-link: geometry collision mesh filename=obj/shoulder.006.obj scale=0.1 0.1 0.1; visual mesh filename=obj/shoulder.003.obj scale=0.1 0.1 0.1
